File: hardware/µ-USBasp_v1.2.brd (EAGLE design)
At the start: 25.4 x 17.8 mm, 15 parts, among them U6 Tiny85-20-SMT

Commit message: Board v1.2
Routing:
- net PB1: track 11.9 -> 13.3 mm
- net PB2: track 16.1 -> 14.8 mm
- net N$2: track 10.1 -> 11.0 mm
Other:
- board size 25.4 x 17.8 mm -> 25.4 x 15.2 mm
- board text added: "GND"
- board text added: "MISO"
- board text added: "MOSI"
- board text added: "NC"
- board text added: "RST"
- board text added: "SCK"
- board text added: "VCC"
